File: Schematic/LDC1000.kicad_sch (KiCad schematic)
At the start: 22 parts, among them IC1 LDC1101DRCT, SW1 SW_DIP_x01, SW2 SW_Push, U1 LM2596S-3.3, U2 ESP32-WROOM-32

Commit message: add button to start detection
Parts:
- added SW3: SW_Push, symbol Switch:SW_Push
Connections:
- net GND: now also SW3.2
- net N_DETECT: now reaches U2.11 (IO26)
- net N_DETECT: now also SW3.1
- no-connect marks 21 -> 20
Changed lines of the file:
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@@
   (no_connect (at 159.258 96.012))
   (no_connect (at 128.778 118.872))
-  (no_connect (at 159.258 131.572))
   (no_connect (at 159.258 126.492))
   (no_connect (at 237.744 107.696))
@@
     (stroke (width 0) (type default))
   )
+  (wire (pts (xy 179.07 131.572) (xy 179.07 133.858))
+    (stroke (width 0) (type default))
+  )
   (wire (pts (xy 32.512 102.616) (xy 32.512 111.506))
     (stroke (width 0) (type default))
@@
     (stroke (width 0) (type default))
   )
+  (wire (pts (xy 159.258 131.572) (xy 179.07 131.572))
+    (stroke (width 0) (type default))
+  )
   (wire (pts (xy 21.082 106.426) (xy 21.082 111.506))
     (stroke (width 0) (type default))
@@
     (stroke (width 0) (type default))
   )
+  (wire (pts (xy 179.07 144.018) (xy 179.07 147.828))
+    (stroke (width 0) (type default))
+  )
   (wire (pts (xy 175.006 90.932) (xy 179.578 90.932))
     (stroke (width 0) (type default))
@@
   )
   (label "PROGRAM" (at 162.052 85.852 0) (fields_autoplaced)
+    (effects (font (size 1.27 1.27)) (justify left bottom))
+  )
+  (label "N_DETECT" (at 169.672 131.572 0) (fields_autoplaced)
     (effects (font (size 1.27 1.27)) (justify left bottom))
   )
@@
     )
   )
+  (symbol (lib_id "power:GND") (at 179.07 147.828 0) (unit 1)
+    (in_bom yes) (on_board yes) (dnp no) (fields_autoplaced)
+    (property "Reference" "#PWR021" (at 179.07 154.178 0)
+      (effects (font (size 1.27 1.27)) hide)
+    )
+    (property "Value" "GND" (at 179.07 152.908 0)
+      (effects (font (size 1.27 1.27)) hide)
+    )
+    (property "Footprint" "" (at 179.07 147.828 0)
+      (effects (font (size 1.27 1.27)) hide)
+    )
+    (property "Datasheet" "" (at 179.07 147.828 0)
+      (effects (font (size 1.27 1.27)) hide)
+    )
+    (pin "1")
+    (instances
+      (project "LDC1000"
+        (path "/c9bb4ff0-f433-4f85-aa38-9b433a61b4bd"
+          (reference "#PWR021") (unit 1)
+        )
+      )
+    )
+  )
   (symbol (lib_id "power:GND") (at 153.162 72.39 90) (unit 1)
     (in_bom yes) (on_board yes) (dnp no) (fields_autoplaced)
@@
         )
       )
+    )
+  )
+  (symbol (lib_id "Switch:SW_Push") (at 179.07 138.938 270) (unit 1)
+    (in_bom yes) (on_board yes) (dnp no) (fields_autoplaced)
+    (property "Reference" "SW3" (at 182.88 138.303 90)
+      (effects (font (size 1.27 1.27)) (justify left))
+    )
+    (property "Value" "SW_Push" (at 182.88 140.843 90)
+      (effects (font (size 1.27 1.27)) (justify left))
+    )
+    (property "Footprint" "" (at 184.15 138.938 0)
+      (effects (font (size 1.27 1.27)) hide)
+    )
+    (property "Datasheet" "~" (at 184.15 138.938 0)
+      (effects (font (size 1.27 1.27)) hide)
+    )
+    (pin "1")
+    (pin "2")
+    (instances
+      (project "LDC1000"
+        (path "/c9bb4ff0-f433-4f85-aa38-9b433a61b4bd"
+          (reference "SW3") (unit 1)
+        )
+      )

Commit message: update firmware
Connections:
- net CLKIN: now also U2.26 (IO4); no longer U2.8 (IO32)
Changed lines of the file:
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@@
   (no_connect (at 159.258 123.952))
   (no_connect (at 128.778 121.412))
-  (no_connect (at 159.258 96.012))
+  (no_connect (at 159.258 136.652))
   (no_connect (at 128.778 118.872))
   (no_connect (at 159.258 126.492))
@@
     (stroke (width 0) (type default))
   )
-  (wire (pts (xy 159.258 136.652) (xy 165.1 136.652))
+  (wire (pts (xy 159.258 96.012) (xy 165.1 96.012))
     (stroke (width 0) (type default))
   )
@@
     )
   )
-  (global_label "CLKIN" (shape input) (at 165.1 136.652 0) (fields_autoplaced)
+  (global_label "CLKIN" (shape input) (at 165.1 96.012 0) (fields_autoplaced)
     (effects (font (size 1.27 1.27)) (justify left))
-    (property "Intersheetrefs" "${INTERSHEET_REFS}" (at 173.5092 136.652 0)
+    (property "Intersheetrefs" "${INTERSHEET_REFS}" (at 173.5092 96.012 0)
       (effects (font (size 1.27 1.27)) (justify left) hide)
     )

Commit message: fix current voltage regulator
Other:
- note added: "12V / 3.3V 2A"
- note removed: "12V / 3.3V 5A"
Changed lines of the file:
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@@
     (effects (font (size 1.27 1.27) bold) (justify left bottom))
   )
-  (text "12V / 3.3V 5A" (at 14.732 119.126 0)
+  (text "12V / 3.3V 2A" (at 14.732 119.126 0)
     (effects (font (size 1.27 1.27) bold) (justify left bottom))
   )
